Commit message: Update tetraDS.xacro

File: tetraDS_description/urdf/tetraDS/tetraDS.xacro (robot description, xacro)
@@ -103,4 +103,5 @@
     <child link="camera1_link" />
   </joint>
+<!--
    <link name="camera2_link">
       <visual>
@@ -111,11 +112,12 @@
         <material name="Grey" />
       </visual>
-  </link>
-  <joint name="camera2_link" type="fixed">
-    <!--<origin xyz="0.1553 -0.1155 0.0" rpy="3.14 -0.261799 0" />-->
+  </link> 240314 -->
+<!--
+  <joint name="camera2_link" type="fixed"> -->
+    <!--<origin xyz="0.1553 -0.1155 0.0" rpy="3.14 -0.261799 0" />--> <!--
     <origin xyz="-0.3118 0.0 0.1985" rpy="0 0 ${PI}" />
     <parent link="base_link"/>
     <child link="camera2_link" />
-  </joint>
+  </joint>-->
  <link name="base_Upperlink">
    <visual>

Commit message: Update tetraDS.xacro

File: tetraDS_description/urdf/tetraDS/tetraDS.xacro (robot description, xacro)
@@ -103,5 +103,4 @@
     <child link="camera1_link" />
   </joint>
-<!--
    <link name="camera2_link">
       <visual>
@@ -112,12 +111,11 @@
         <material name="Grey" />
       </visual>
-  </link> 240314 -->
-<!--
-  <joint name="camera2_link" type="fixed"> -->
-    <!--<origin xyz="0.1553 -0.1155 0.0" rpy="3.14 -0.261799 0" />--> <!--
+  </link>
+  <joint name="camera2_link" type="fixed">
+    <!--<origin xyz="0.1553 -0.1155 0.0" rpy="3.14 -0.261799 0" />-->
     <origin xyz="-0.3118 0.0 0.1985" rpy="0 0 ${PI}" />
     <parent link="base_link"/>
     <child link="camera2_link" />
-  </joint>-->
+  </joint>
  <link name="base_Upperlink">
    <visual>

Commit message: Update tetraDS.xacro

File: tetraDS_description/urdf/tetraDS/tetraDS.xacro (robot description, xacro)
@@ -88,19 +88,5 @@
     <child link="Front_bumper" />
   </joint>
- <link name="camera1_link">
-      <visual>
-        <origin xyz="0 0 0" rpy="0 0 0" />
-        <geometry>
-          <box size="0.01 0.01 0.01" />
-        </geometry>
-        <material name="Grey" />
-      </visual>
-  </link>
-  <joint name="camera1_link" type="fixed">
-    <!--<origin xyz="0.1553 -0.1155 0.0" rpy="3.14 -0.261799 0" />-->
-    <origin xyz="0.1347 0.0 0.1344" rpy="0 0 0" />
-    <parent link="base_link"/>
-    <child link="camera1_link" />
-  </joint>
+<!-- 240314 mwcha Removed 'camera1_link' because S model just have a single depth camera -->
    <link name="camera2_link">
       <visual>
@@ -114,5 +100,5 @@
   <joint name="camera2_link" type="fixed">
     <!--<origin xyz="0.1553 -0.1155 0.0" rpy="3.14 -0.261799 0" />-->
-    <origin xyz="-0.3118 0.0 0.1985" rpy="0 0 ${PI}" />
+    <origin xyz="0.1347 0.0 0.1344" rpy="0 0 0" />
     <parent link="base_link"/>
     <child link="camera2_link" />
